File: Hardware/Driver.kicad_sch (KiCad schematic)
At the start: 27 parts, among them J1 Motor, U1 MP6540

Commit message: 小修小补，拉了点线
Parts:
- removed R19: 0R, myDevice:0603_R, symbol Device:R
- removed TP1, TP2, TP3, TP4: TestPoint, TestPoint:TestPoint_Pad_D1.0mm, symbol Connector:TestPoint
Other:
- company: Akako Industry -> Akako Science & Industry
Changed lines of the file:
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@@
     (date "2023-03-19")
     (rev "1.0")
-    (company "Akako Industry")
+    (company "Akako Science & Industry")
     (comment 1 "赤紫绮")
     (comment 2 "赤紫绮")
@@
   (junction (at 238.76 86.36) (diameter 0) (color 0 0 0 0)
   )
-  (junction (at 128.27 57.15) (diameter 0) (color 0 0 0 0)
-  )
   (junction (at 90.17 63.5) (diameter 0) (color 0 0 0 0)
   )
   (junction (at 172.72 100.33) (diameter 0) (color 0 0 0 0)
   )
-  (junction (at 138.43 110.49) (diameter 0) (color 0 0 0 0)
-  )
   (junction (at 137.16 77.47) (diameter 0) (color 0 0 0 0)
   )
   (junction (at 73.66 115.57) (diameter 0) (color 0 0 0 0)
   )
-  (junction (at 120.65 63.5) (diameter 0) (color 0 0 0 0)
-  )
   (junction (at 120.65 100.33) (diameter 0) (color 0 0 0 0)
   )
-  (junction (at 163.83 110.49) (diameter 0) (color 0 0 0 0)
-  )
   (junction (at 238.76 99.06) (diameter 0) (color 0 0 0 0)
   )
@@
   (junction (at 120.65 115.57) (diameter 0) (color 0 0 0 0)
   )
-  (junction (at 113.03 69.85) (diameter 0) (color 0 0 0 0)
-  )
   (junction (at 128.27 97.79) (diameter 0) (color 0 0 0 0)
   )
@@
     (stroke (width 0) (type default))
   )
-  (wire (pts (xy 154.94 110.49) (xy 163.83 110.49))
-    (stroke (width 0) (type default))
-  )
   (wire (pts (xy 238.76 88.9) (xy 238.76 86.36))
     (stroke (width 0) (type default))
@@
     (stroke (width 0) (type default))
   )
-  (wire (pts (xy 113.03 40.64) (xy 113.03 69.85))
-    (stroke (width 0) (type default))
-  )
   (wire (pts (xy 109.22 57.15) (xy 128.27 57.15))
     (stroke (width 0) (type default))
@@
     (stroke (width 0) (type default))
   )
-  (wire (pts (xy 133.35 40.64) (xy 113.03 40.64))
-    (stroke (width 0) (type default))
-  )
-  (wire (pts (xy 163.83 110.49) (xy 163.83 113.03))
+  (wire (pts (xy 163.83 105.41) (xy 163.83 113.03))
     (stroke (width 0) (type default))
   )
@@
     (stroke (width 0) (type default))
   )
-  (wire (pts (xy 133.35 50.8) (xy 128.27 50.8))
-    (stroke (width 0) (type default))
-  )
   (wire (pts (xy 161.29 86.36) (xy 228.6 86.36))
     (stroke (width 0) (type default))
@@
     (stroke (width 0) (type default))
   )
-  (wire (pts (xy 163.83 105.41) (xy 163.83 110.49))
-    (stroke (width 0) (type default))
-  )
-  (wire (pts (xy 128.27 50.8) (xy 128.27 57.15))
-    (stroke (width 0) (type default))
-  )
   (wire (pts (xy 109.22 63.5) (xy 120.65 63.5))
     (stroke (width 0) (type default))
   )
-  (wire (pts (xy 138.43 110.49) (xy 147.32 110.49))
-    (stroke (width 0) (type default))
-  )
   (wire (pts (xy 104.14 77.47) (xy 137.16 77.47))
     (stroke (width 0) (type default))
@@
     (stroke (width 0) (type default))
   )
-  (wire (pts (xy 120.65 45.72) (xy 120.65 63.5))
-    (stroke (width 0) (type default))
-  )
   (wire (pts (xy 113.03 113.03) (xy 113.03 115.57))
     (stroke (width 0) (type default))
@@
     (stroke (width 0) (type default))
   )
-  (wire (pts (xy 138.43 110.49) (xy 138.43 113.03))
+  (wire (pts (xy 138.43 105.41) (xy 138.43 113.03))
     (stroke (width 0) (type default))
   )
@@
     (stroke (width 0) (type default))
   )
-  (wire (pts (xy 133.35 45.72) (xy 120.65 45.72))
-    (stroke (width 0) (type default))
-  )
   (wire (pts (xy 120.65 115.57) (xy 128.27 115.57))
-    (stroke (width 0) (type default))
-  )
-  (wire (pts (xy 138.43 105.41) (xy 138.43 110.49))
     (stroke (width 0) (type default))
   )
@@
     (effects (font (size 1.27 1.27)) (justify left bottom))
   )
-  (label "VMOTOR" (at 163.83 88.9 0) (fields_autoplaced)
+  (label "VIN" (at 163.83 88.9 0) (fields_autoplaced)
     (effects (font (size 1.27 1.27)) (justify left bottom))
   )
@@
     )
   )
-  (symbol (lib_id "Connector:TestPoint") (at 133.35 35.56 270) (unit 1)
-    (in_bom yes) (on_board yes) (dnp no) (fields_autoplaced)
-    (property "Reference" "TP4" (at 138.43 34.925 90)
-      (effects (font (size 1.27 1.27)) (justify left))
-    )
-    (property "Value" "TestPoint" (at 138.43 37.465 90)
-      (effects (font (size 1.27 1.27)) (justify left))
-    )
-    (property "Footprint" "TestPoint:TestPoint_Pad_D1.0mm" (at 133.35 40.64 0)
-      (effects (font (size 1.27 1.27)) hide)
-    )
-    (property "Datasheet" "~" (at 133.35 40.64 0)
-      (effects (font (size 1.27 1.27)) hide)
-    )
-    (pin "1")
-    (instances
-      (project "cwFOC"
-        (path "/ff847474-9801-42c6-af12-b4b1b75aa0af/c3a6c5b4-78f3-47ea-a70d-c3f42438cf04"
-          (reference "TP4") (unit 1)
-        )
-      )
-    )
-  )
   (symbol (lib_id "power:+3V3") (at 137.16 67.31 0) (unit 1)
     (in_bom yes) (on_board yes) (dnp no) (fields_autoplaced)
@@
         (path "/ff847474-9801-42c6-af12-b4b1b75aa0af/c3a6c5b4-78f3-47ea-a70d-c3f42438cf04"
           (reference "#PWR047") (unit 1)
-        )
-      )
-    )
-  )
-  (symbol (lib_id "Connector:TestPoint") (at 133.35 40.64 270) (unit 1)
-    (in_bom yes) (on_board yes) (dnp no) (fields_autoplaced)
-    (property "Reference" "TP1" (at 138.43 40.005 90)
-      (effects (font (size 1.27 1.27)) (justify left))
-    )
-    (property "Value" "TestPoint" (at 138.43 42.545 90)
-      (effects (font (size 1.27 1.27)) (justify left))
-    )
-    (property "Footprint" "TestPoint:TestPoint_Pad_D1.0mm" (at 133.35 45.72 0)
-      (effects (font (size 1.27 1.27)) hide)
-    )
-    (property "Datasheet" "~" (at 133.35 45.72 0)
-      (effects (font (size 1.27 1.27)) hide)
-    )
-    (pin "1")
-    (instances
-      (project "cwFOC"
-        (path "/ff847474-9801-42c6-af12-b4b1b75aa0af/c3a6c5b4-78f3-47ea-a70d-c3f42438cf04"
-          (reference "TP1") (unit 1)
         )
       )
@@
     )
   )
-  (symbol (lib_id "Device:R") (at 151.13 110.49 90) (unit 1)
-    (in_bom yes) (on_board yes) (dnp no) (fields_autoplaced)
-    (property "Reference" "R19" (at 151.13 114.3 90)
-      (effects (font (size 1.27 1.27)))
-    )
-    (property "Value" "0R" (at 151.13 116.84 90)
-      (effects (font (size 1.27 1.27)))
-    )
-    (property "Footprint" "myDevice:0603_R" (at 151.13 112.268 90)
-      (effects (font (size 1.27 1.27)) hide)
-    )
-    (property "Datasheet" "~" (at 151.13 110.49 0)
-      (effects (font (size 1.27 1.27)) hide)
-    )
-    (pin "1")
-    (pin "2")
-    (instances
-      (project "cwFOC"
-        (path "/ff847474-9801-42c6-af12-b4b1b75aa0af/c3a6c5b4-78f3-47ea-a70d-c3f42438cf04"
-          (reference "R19") (unit 1)
-        )
-      )
-    )
-  )
   (symbol (lib_id "power:GND") (at 90.17 74.93 0) (unit 1)
     (in_bom yes) (on_board yes) (dnp no) (fields_autoplaced)
@@
         (path "/ff847474-9801-42c6-af12-b4b1b75aa0af/c3a6c5b4-78f3-47ea-a70d-c3f42438cf04"
           (reference "#PWR017") (unit 1)
-        )
-      )
-    )
-  )
-  (symbol (lib_id "power:GND") (at 133.35 35.56 270) (unit 1)
-    (in_bom yes) (on_board yes) (dnp no) (fields_autoplaced)
-    (property "Reference" "#PWR015" (at 127 35.56 0)
-      (effects (font (size 1.27 1.27)) hide)
-    )
-    (property "Value" "GND" (at 129.54 36.195 90)
-      (effects (font (size 1.27 1.27)) (justify right))
-    )
-    (property "Footprint" "" (at 133.35 35.56 0)
-      (effects (font (size 1.27 1.27)) hide)
-    )
-    (property "Datasheet" "" (at 133.35 35.56 0)
-      (effects (font (size 1.27 1.27)) hide)
-    )
-    (pin "1")
-    (instances
-      (project "cwFOC"
-        (path "/ff847474-9801-42c6-af12-b4b1b75aa0af/c3a6c5b4-78f3-47ea-a70d-c3f42438cf04"
-          (reference "#PWR015") (unit 1)
         )
       )
@@
     )
   )
-  (symbol (lib_id "Connector:TestPoint") (at 133.35 50.8 270) (unit 1)
-    (in_bom yes) (on_board yes) (dnp no) (fields_autoplaced)
-    (property "Reference" "TP3" (at 138.43 50.165 90)
-      (effects (font (size 1.27 1.27)) (justify left))
-    )
-    (property "Value" "TestPoint" (at 138.43 52.705 90)
-      (effects (font (size 1.27 1.27)) (justify left))
-    )
-    (property "Footprint" "TestPoint:TestPoint_Pad_D1.0mm" (at 133.35 55.88 0)
-      (effects (font (size 1.27 1.27)) hide)
-    )
-    (property "Datasheet" "~" (at 133.35 55.88 0)
-      (effects (font (size 1.27 1.27)) hide)
-    )
-    (pin "1")
-    (instances
-      (project "cwFOC"
-        (path "/ff847474-9801-42c6-af12-b4b1b75aa0af/c3a6c5b4-78f3-47ea-a70d-c3f42438cf04"
-          (reference "TP3") (unit 1)
-        )
-      )
-    )
-  )
   (symbol (lib_id "Device:C_Small") (at 168.91 80.01 180) (unit 1)
     (in_bom yes) (on_board yes) (dnp no) (fields_autoplaced)
@@
         )
       )
-    )
-  )
-  (symbol (lib_id "Connector:TestPoint") (at 133.35 45.72 270) (unit 1)
-    (in_bom yes) (on_board yes) (dnp no) (fields_autoplaced)
-    (property "Reference" "TP2" (at 138.43 45.085 90)
-      (effects (font (size 1.27 1.27)) (justify left))
-    )
-    (property "Value" "TestPoint" (at 138.43 47.625 90)
-      (effects (font (size 1.27 1.27)) (justify left))
-    )
-    (property "Footprint" "TestPoint:TestPoint_Pad_D1.0mm" (at 133.35 50.8 0)
-      (effects (font (size 1.27 1.27)) hide)
-    )
-    (property "Datasheet" "~" (at 133.35 50.8 0)
-      (effects (font (size 1.27 1.27)) hide)
-    )
-    (pin "1")
-    (instances
-      (project "cwFOC"
-        (path "/ff847474-9801-42c6-af12-b4b1b75aa0af/c3a6c5b4-78f3-47ea-a70d-c3f42438cf04"
-          (reference "TP2") (unit 1)
-        )
-      )
