File: Hardware/Encoder.kicad_sch (KiCad schematic)
At the start: 7 parts, among them U2 AS5600

Commit message: 完成原理图设计，完成初步布局布线
Parts:
- removed C6: 0.1uF, myDevice:0603_C, symbol Device:C
- removed R3: 0R, myDevice:0603_R, symbol Device:R
Connections:
- net +3V3: now also C6.2, U2.2 (VDD3V3)
Changed lines of the file:
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@@
 (kicad_sch (version 20230121) (generator eeschema)
   (paper "A4")
-  (junction (at 107.95 91.44) (diameter 0) (color 0 0 0 0)
-  )
-  (junction (at 107.95 99.06) (diameter 0) (color 0 0 0 0)
+  (junction (at 107.95 96.52) (diameter 0) (color 0 0 0 0)
+  )
+  (junction (at 107.95 93.98) (diameter 0) (color 0 0 0 0)
   )
   (junction (at 167.64 83.82) (diameter 0) (color 0 0 0 0)
@@
     (stroke (width 0) (type default))
   )
-  (wire (pts (xy 107.95 91.44) (xy 107.95 93.98))
-    (stroke (width 0) (type default))
-  )
   (wire (pts (xy 168.91 86.36) (xy 168.91 83.82))
     (stroke (width 0) (type default))
@@
     (stroke (width 0) (type default))
   )
-  (wire (pts (xy 102.87 91.44) (xy 107.95 91.44))
-    (stroke (width 0) (type default))
-  )
   (wire (pts (xy 154.94 101.6) (xy 154.94 104.14))
     (stroke (width 0) (type default))
@@
     (stroke (width 0) (type default))
   )
-  (wire (pts (xy 102.87 99.06) (xy 107.95 99.06))
-    (stroke (width 0) (type default))
-  )
-  (wire (pts (xy 107.95 96.52) (xy 107.95 99.06))
-    (stroke (width 0) (type default))
-  )
   (wire (pts (xy 166.37 83.82) (xy 167.64 83.82))
     (stroke (width 0) (type default))
@@
     (stroke (width 0) (type default))
   )
-  (wire (pts (xy 107.95 99.06) (xy 107.95 101.6))
-    (stroke (width 0) (type default))
-  )
-  (wire (pts (xy 107.95 90.17) (xy 107.95 91.44))
+  (wire (pts (xy 107.95 93.98) (xy 107.95 96.52))
+    (stroke (width 0) (type default))
+  )
+  (wire (pts (xy 107.95 90.17) (xy 107.95 93.98))
+    (stroke (width 0) (type default))
+  )
+  (wire (pts (xy 107.95 96.52) (xy 107.95 101.6))
     (stroke (width 0) (type default))
   )
@@
   (hierarchical_label "SDA" (shape bidirectional) (at 176.53 99.06 0) (fields_autoplaced)
     (effects (font (size 1.27 1.27)) (justify left))
-  )
-  (symbol (lib_id "Device:C") (at 118.11 77.47 180) (unit 1)
-    (in_bom yes) (on_board yes) (dnp no) (fields_autoplaced)
-    (property "Reference" "C6" (at 121.92 76.835 0)
-      (effects (font (size 1.27 1.27)) (justify right))
-    )
-    (property "Value" "0.1uF" (at 121.92 79.375 0)
-      (effects (font (size 1.27 1.27)) (justify right))
-    )
-    (property "Footprint" "myDevice:0603_C" (at 117.1448 73.66 0)
-      (effects (font (size 1.27 1.27)) hide)
-    )
-    (property "Datasheet" "~" (at 118.11 77.47 0)
-      (effects (font (size 1.27 1.27)) hide)
-    )
-    (pin "1")
-    (pin "2")
-    (instances
-      (project "cwFOC"
-        (path "/ff847474-9801-42c6-af12-b4b1b75aa0af"
-          (reference "C6") (unit 1)
-        )
-        (path "/ff847474-9801-42c6-af12-b4b1b75aa0af/dedc76e1-245b-4c26-9dc4-835534115ef4"
-          (reference "C4") (unit 1)
-        )
-      )
-    )
   )
   (symbol (lib_id "power:GND") (at 134.62 101.6 270) (unit 1)
@@
     )
   )
-  (symbol (lib_id "power:GND") (at 118.11 81.28 0) (unit 1)
-    (in_bom yes) (on_board yes) (dnp no) (fields_autoplaced)
-    (property "Reference" "#PWR011" (at 118.11 87.63 0)
-      (effects (font (size 1.27 1.27)) hide)
-    )
-    (property "Value" "GND" (at 118.11 86.36 0)
-      (effects (font (size 1.27 1.27)))
-    )
-    (property "Footprint" "" (at 118.11 81.28 0)
-      (effects (font (size 1.27 1.27)) hide)
-    )
-    (property "Datasheet" "" (at 118.11 81.28 0)
+  (symbol (lib_id "power:GND") (at 107.95 109.22 0) (unit 1)
+    (in_bom yes) (on_board yes) (dnp no) (fields_autoplaced)
+    (property "Reference" "#PWR011" (at 107.95 115.57 0)
+      (effects (font (size 1.27 1.27)) hide)
+    )
+    (property "Value" "GND" (at 107.95 114.3 0)
+      (effects (font (size 1.27 1.27)))
+    )
+    (property "Footprint" "" (at 107.95 109.22 0)
+      (effects (font (size 1.27 1.27)) hide)
+    )
+    (property "Datasheet" "" (at 107.95 109.22 0)
       (effects (font (size 1.27 1.27)) hide)
     )
@@
         )
         (path "/ff847474-9801-42c6-af12-b4b1b75aa0af/dedc76e1-245b-4c26-9dc4-835534115ef4"
-          (reference "#PWR031") (unit 1)
-        )
-      )
-    )
-  )
-  (symbol (lib_id "power:GND") (at 107.95 109.22 0) (unit 1)
-    (in_bom yes) (on_board yes) (dnp no) (fields_autoplaced)
-    (property "Reference" "#PWR011" (at 107.95 115.57 0)
-      (effects (font (size 1.27 1.27)) hide)
-    )
-    (property "Value" "GND" (at 107.95 114.3 0)
-      (effects (font (size 1.27 1.27)))
-    )
-    (property "Footprint" "" (at 107.95 109.22 0)
-      (effects (font (size 1.27 1.27)) hide)
-    )
-    (property "Datasheet" "" (at 107.95 109.22 0)
-      (effects (font (size 1.27 1.27)) hide)
-    )
-    (pin "1")
-    (instances
-      (project "cwFOC"
-        (path "/ff847474-9801-42c6-af12-b4b1b75aa0af"
-          (reference "#PWR011") (unit 1)
-        )
-        (path "/ff847474-9801-42c6-af12-b4b1b75aa0af/dedc76e1-245b-4c26-9dc4-835534115ef4"
           (reference "#PWR09") (unit 1)
-        )
-      )
-    )
-  )
-  (symbol (lib_id "Device:R") (at 102.87 95.25 180) (unit 1)
-    (in_bom yes) (on_board yes) (dnp no) (fields_autoplaced)
-    (property "Reference" "R3" (at 100.33 94.615 0)
-      (effects (font (size 1.27 1.27)) (justify left))
-    )
-    (property "Value" "0R" (at 100.33 97.155 0)
-      (effects (font (size 1.27 1.27)) (justify left))
-    )
-    (property "Footprint" "myDevice:0603_R" (at 104.648 95.25 90)
-      (effects (font (size 1.27 1.27)) hide)
-    )
-    (property "Datasheet" "~" (at 102.87 95.25 0)
-      (effects (font (size 1.27 1.27)) hide)
-    )
-    (pin "1")
-    (pin "2")
-    (instances
-      (project "cwFOC"
-        (path "/ff847474-9801-42c6-af12-b4b1b75aa0af"
-          (reference "R3") (unit 1)
-        )
-        (path "/ff847474-9801-42c6-af12-b4b1b75aa0af/dedc76e1-245b-4c26-9dc4-835534115ef4"
-          (reference "R10") (unit 1)
         )
       )
@@
         )
       )
-    )
-  )
-  (symbol (lib_id "power:+3V3") (at 118.11 73.66 0) (unit 1)
-    (in_bom yes) (on_board yes) (dnp no) (fields_autoplaced)
-    (property "Reference" "#PWR032" (at 118.11 77.47 0)
-      (effects (font (size 1.27 1.27)) hide)
-    )
-    (property "Value" "+3V3" (at 118.11 69.85 0)
-      (effects (font (size 1.27 1.27)))
-    )
-    (property "Footprint" "" (at 118.11 73.66 0)
-      (effects (font (size 1.27 1.27)) hide)
-    )
-    (property "Datasheet" "" (at 118.11 73.66 0)
-      (effects (font (size 1.27 1.27)) hide)
-    )
-    (pin "1")
-    (instances
-      (project "cwFOC"
-        (path "/ff847474-9801-42c6-af12-b4b1b75aa0af/dedc76e1-245b-4c26-9dc4-835534115ef4"
-          (reference "#PWR032") (unit 1)
-        )
-      )

Commit message: 基本完成PCB设计
Parts:
- U2: footprint Package_SO:SOP-8_3.9x4.9mm_P1.27mm -> Package_SO:SOIC-8_3.9x4.9mm_P1.27mm
Changed lines of the file:
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@@
       (effects (font (size 1.27 1.27)))
     )
-    (property "Footprint" "Package_SO:SOP-8_3.9x4.9mm_P1.27mm" (at 143.51 106.68 0)
+    (property "Footprint" "Package_SO:SOIC-8_3.9x4.9mm_P1.27mm" (at 143.51 106.68 0)
       (effects (font (size 1.27 1.27)) hide)
     )

Commit message: 第一版硬件做好啦！(●'◡'●)
Other:
- company: (none) -> Akako Industry
- title: (none) -> cwFOC/Encoder
Changed lines of the file:
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@@
 (kicad_sch (version 20230121) (generator eeschema)
   (paper "A4")
+  (title_block
+    (title "cwFOC/Encoder")
+    (date "2023-03-19")
+    (rev "1.0")
+    (company "Akako Industry")
+    (comment 1 "赤紫绮")
+    (comment 2 "赤紫绮")
+    (comment 3 "赤紫绮")
+  )
   (junction (at 107.95 96.52) (diameter 0) (color 0 0 0 0)
   )

Commit message: 小修小补，拉了点线
Parts:
- removed R4: 0R, myDevice:0603_R, symbol Device:R
Connections:
- no-connect marks 0 -> 1
Other:
- company: Akako Industry -> Akako Science & Industry
Changed lines of the file:
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@@
     (date "2023-03-19")
     (rev "1.0")
-    (company "Akako Industry")
+    (company "Akako Science & Industry")
     (comment 1 "赤紫绮")
     (comment 2 "赤紫绮")
@@
   (junction (at 166.37 99.06) (diameter 0) (color 0 0 0 0)
   )
+  (no_connect (at 152.4 101.6))
   (wire (pts (xy 168.91 93.98) (xy 168.91 96.52))
     (stroke (width 0) (type default))
@@
   )
   (wire (pts (xy 166.37 86.36) (xy 166.37 83.82))
-    (stroke (width 0) (type default))
-  )
-  (wire (pts (xy 154.94 101.6) (xy 154.94 104.14))
-    (stroke (width 0) (type default))
-  )
-  (wire (pts (xy 152.4 101.6) (xy 154.94 101.6))
     (stroke (width 0) (type default))
   )
@@
     )
   )
-  (symbol (lib_id "power:GND") (at 154.94 111.76 0) (unit 1)
-    (in_bom yes) (on_board yes) (dnp no) (fields_autoplaced)
-    (property "Reference" "#PWR013" (at 154.94 118.11 0)
-      (effects (font (size 1.27 1.27)) hide)
-    )
-    (property "Value" "GND" (at 154.94 116.84 0)
-      (effects (font (size 1.27 1.27)))
-    )
-    (property "Footprint" "" (at 154.94 111.76 0)
-      (effects (font (size 1.27 1.27)) hide)
-    )
-    (property "Datasheet" "" (at 154.94 111.76 0)
-      (effects (font (size 1.27 1.27)) hide)
-    )
-    (pin "1")
-    (instances
-      (project "cwFOC"
-        (path "/ff847474-9801-42c6-af12-b4b1b75aa0af"
-          (reference "#PWR013") (unit 1)
-        )
-        (path "/ff847474-9801-42c6-af12-b4b1b75aa0af/dedc76e1-245b-4c26-9dc4-835534115ef4"
-          (reference "#PWR013") (unit 1)
-        )
-      )
-    )
-  )
   (symbol (lib_id "Device:C") (at 107.95 105.41 180) (unit 1)
     (in_bom yes) (on_board yes) (dnp no) (fields_autoplaced)
@@
         )
       )
-    )
-  )
-  (symbol (lib_id "Device:R") (at 154.94 107.95 180) (unit 1)
-    (in_bom no) (on_board yes) (dnp yes) (fields_autoplaced)
-    (property "Reference" "R4" (at 157.48 106.68 0)
-      (effects (font (size 1.27 1.27)) (justify right))
-    )
-    (property "Value" "0R" (at 157.48 109.22 0)
-      (effects (font (size 1.27 1.27)) (justify right))
-    )
-    (property "Footprint" "myDevice:0603_R" (at 156.718 107.95 90)
-      (effects (font (size 1.27 1.27)) hide)
-    )
-    (property "Datasheet" "~" (at 154.94 107.95 0)
-      (effects (font (size 1.27 1.27)) hide)
-    )
-    (pin "1")
-    (pin "2")
-    (instances
-      (project "cwFOC"
-        (path "/ff847474-9801-42c6-af12-b4b1b75aa0af"
-          (reference "R4") (unit 1)
-        )
-        (path "/ff847474-9801-42c6-af12-b4b1b75aa0af/dedc76e1-245b-4c26-9dc4-835534115ef4"
-          (reference "R2") (unit 1)
-        )
-      )

Commit message: 完成第二版硬件
Parts:
- R2, R3: value 4.7K -> 2.2K
Changed lines of the file:
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@@
       (effects (font (size 1.27 1.27)) (justify right))
     )
-    (property "Value" "4.7K" (at 171.45 92.075 0)
+    (property "Value" "2.2K" (at 171.45 92.075 0)
       (effects (font (size 1.27 1.27)) (justify right))
     )
@@
       (effects (font (size 1.27 1.27)) (justify left))
     )
-    (property "Value" "4.7K" (at 163.83 92.075 0)
+    (property "Value" "2.2K" (at 163.83 92.075 0)
       (effects (font (size 1.27 1.27)) (justify left))
     )
