File: Hardware/RS485.kicad_sch (KiCad schematic)
At the start: 6 parts, among them J3 KF2EDGV, U2 MAX3485

Commit message: 基本完成PCB设计
Connections:
- net GND: no longer J3.5 (Pin_5)
- new net GNDPWR: J3.5 (Pin_5)
Changed lines of the file:
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@@
+    (stroke (width 0) (type default))
+  )
+  (wire (pts (xy 182.88 133.35) (xy 182.88 138.43))
     (stroke (width 0) (type default))
   )
@@
   (hierarchical_label "RX" (shape output) (at 116.84 87.63 180) (fields_autoplaced)
     (effects (font (size 1.27 1.27)) (justify right))
-  )
-  (symbol (lib_id "power:GND") (at 182.88 133.35 270) (unit 1)
-    (in_bom yes) (on_board yes) (dnp no) (fields_autoplaced)
-    (property "Reference" "#PWR031" (at 176.53 133.35 0)
-      (effects (font (size 1.27 1.27)) hide)
-    )
-    (property "Value" "GND" (at 179.07 133.985 90)
-      (effects (font (size 1.27 1.27)) (justify right))
-    )
-    (property "Footprint" "" (at 182.88 133.35 0)
-      (effects (font (size 1.27 1.27)) hide)
-    )
-    (property "Datasheet" "" (at 182.88 133.35 0)
-      (effects (font (size 1.27 1.27)) hide)
-    )
-    (pin "1")
-    (instances
-      (project "cwFOC"
-        (path "/ff847474-9801-42c6-af12-b4b1b75aa0af/50c76e34-9c76-4785-b3ad-3791bfa1e28e"
-          (reference "#PWR031") (unit 1)
-        )
-      )
-    )
   )
   (symbol (lib_id "power:GND") (at 140.97 105.41 0) (unit 1)
@@
         )
       )
+    )
+  )
+  (symbol (lib_id "power:GNDPWR") (at 182.88 138.43 0) (unit 1)
+    (in_bom yes) (on_board yes) (dnp no) (fields_autoplaced)
+    (property "Reference" "#PWR031" (at 182.88 143.51 0)
+      (effects (font (size 1.27 1.27)) hide)
+    )
+    (property "Value" "GNDPWR" (at 182.753 143.51 0)
+      (effects (font (size 1.27 1.27)))
+    )
+    (property "Footprint" "" (at 182.88 139.7 0)
+      (effects (font (size 1.27 1.27)) hide)
+    )
+    (property "Datasheet" "" (at 182.88 139.7 0)
+      (effects (font (size 1.27 1.27)) hide)
+    )
+    (pin "1")
+    (instances
+      (project "cwFOC"
+        (path "/ff847474-9801-42c6-af12-b4b1b75aa0af/50c76e34-9c76-4785-b3ad-3791bfa1e28e"
+          (reference "#PWR031") (unit 1)
+        )
+      )

Commit message: 第一版硬件做好啦！(●'◡'●)
Other:
- company: (none) -> Akako Industry
- title: (none) -> cwFOC/RS485
Changed lines of the file:
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@@
 (kicad_sch (version 20230121) (generator eeschema)
   (paper "A4")
+  (title_block
+    (title "cwFOC/RS485")
+    (date "2023-03-19")
+    (rev "1.0")
+    (company "Akako Industry")
+    (comment 1 "赤紫绮")
+    (comment 2 "赤紫绮")
+    (comment 3 "赤紫绮")
+  )
   (junction (at 128.905 91.44) (diameter 0) (color 0 0 0 0)
   )

Commit message: 小修小补，拉了点线
Connections:
- net +5V renamed +3V3
Other:
- company: Akako Industry -> Akako Science & Industry
Changed lines of the file:
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@@
     (date "2023-03-19")
     (rev "1.0")
-    (company "Akako Industry")
+    (company "Akako Science & Industry")
     (comment 1 "赤紫绮")
     (comment 2 "赤紫绮")
@@
     (effects (font (size 1.27 1.27)) (justify right))
   )
+  (symbol (lib_id "power:+3V3") (at 140.97 77.47 0) (unit 1)
+    (in_bom yes) (on_board yes) (dnp no) (fields_autoplaced)
+    (property "Reference" "#PWR029" (at 140.97 81.28 0)
+      (effects (font (size 1.27 1.27)) hide)
+    )
+    (property "Value" "+3V3" (at 140.97 73.66 0)
+      (effects (font (size 1.27 1.27)))
+    )
+    (property "Footprint" "" (at 140.97 77.47 0)
+      (effects (font (size 1.27 1.27)) hide)
+    )
+    (property "Datasheet" "" (at 140.97 77.47 0)
+      (effects (font (size 1.27 1.27)) hide)
+    )
+    (pin "1")
+    (instances
+      (project "cwFOC"
+        (path "/ff847474-9801-42c6-af12-b4b1b75aa0af/50c76e34-9c76-4785-b3ad-3791bfa1e28e"
+          (reference "#PWR029") (unit 1)
+        )
+      )
+    )
+  )
   (symbol (lib_id "power:GND") (at 140.97 105.41 0) (unit 1)
     (in_bom yes) (on_board yes) (dnp no) (fields_autoplaced)
@@
     )
   )
-  (symbol (lib_id "power:+5V") (at 165.1 102.87 180) (unit 1)
-    (in_bom yes) (on_board yes) (dnp no) (fields_autoplaced)
-    (property "Reference" "#PWR02" (at 165.1 99.06 0)
-      (effects (font (size 1.27 1.27)) hide)
-    )
-    (property "Value" "+5V" (at 165.1 107.95 0)
-      (effects (font (size 1.27 1.27)))
-    )
-    (property "Footprint" "" (at 165.1 102.87 0)
-      (effects (font (size 1.27 1.27)) hide)
-    )
-    (property "Datasheet" "" (at 165.1 102.87 0)
-      (effects (font (size 1.27 1.27)) hide)
-    )
-    (pin "1")
-    (instances
-      (project "cwFOC"
-        (path "/ff847474-9801-42c6-af12-b4b1b75aa0af/50c76e34-9c76-4785-b3ad-3791bfa1e28e"
-          (reference "#PWR02") (unit 1)
-        )
-      )
-    )
-  )
   (symbol (lib_id "power:GND") (at 165.1 80.01 180) (unit 1)
     (in_bom yes) (on_board yes) (dnp no) (fields_autoplaced)
@@
         (path "/ff847474-9801-42c6-af12-b4b1b75aa0af/50c76e34-9c76-4785-b3ad-3791bfa1e28e"
           (reference "#PWR038") (unit 1)
-        )
-      )
-    )
-  )
-  (symbol (lib_id "power:+5V") (at 203.2 87.63 0) (unit 1)
-    (in_bom yes) (on_board yes) (dnp no) (fields_autoplaced)
-    (property "Reference" "#PWR044" (at 203.2 91.44 0)
-      (effects (font (size 1.27 1.27)) hide)
-    )
-    (property "Value" "+5V" (at 203.2 83.82 0)
-      (effects (font (size 1.27 1.27)))
-    )
-    (property "Footprint" "" (at 203.2 87.63 0)
-      (effects (font (size 1.27 1.27)) hide)
-    )
-    (property "Datasheet" "" (at 203.2 87.63 0)
-      (effects (font (size 1.27 1.27)) hide)
-    )
-    (pin "1")
-    (instances
-      (project "cwFOC"
-        (path "/ff847474-9801-42c6-af12-b4b1b75aa0af/50c76e34-9c76-4785-b3ad-3791bfa1e28e"
-          (reference "#PWR044") (unit 1)
         )
       )
@@
     )
   )
-  (symbol (lib_id "power:+5V") (at 140.97 77.47 0) (unit 1)
-    (in_bom yes) (on_board yes) (dnp no) (fields_autoplaced)
-    (property "Reference" "#PWR034" (at 140.97 81.28 0)
-      (effects (font (size 1.27 1.27)) hide)
-    )
-    (property "Value" "+5V" (at 140.97 73.66 0)
-      (effects (font (size 1.27 1.27)))
-    )
-    (property "Footprint" "" (at 140.97 77.47 0)
-      (effects (font (size 1.27 1.27)) hide)
-    )
-    (property "Datasheet" "" (at 140.97 77.47 0)
-      (effects (font (size 1.27 1.27)) hide)
-    )
-    (pin "1")
-    (instances
-      (project "cwFOC"
-        (path "/ff847474-9801-42c6-af12-b4b1b75aa0af/50c76e34-9c76-4785-b3ad-3791bfa1e28e"
-          (reference "#PWR034") (unit 1)
+  (symbol (lib_id "power:+3V3") (at 165.1 102.87 180) (unit 1)
+    (in_bom yes) (on_board yes) (dnp no) (fields_autoplaced)
+    (property "Reference" "#PWR02" (at 165.1 99.06 0)
+      (effects (font (size 1.27 1.27)) hide)
+    )
+    (property "Value" "+3V3" (at 165.1 107.95 0)
+      (effects (font (size 1.27 1.27)))
+    )
+    (property "Footprint" "" (at 165.1 102.87 0)
+      (effects (font (size 1.27 1.27)) hide)
+    )
+    (property "Datasheet" "" (at 165.1 102.87 0)
+      (effects (font (size 1.27 1.27)) hide)
+    )
+    (pin "1")
+    (instances
+      (project "cwFOC"
+        (path "/ff847474-9801-42c6-af12-b4b1b75aa0af/50c76e34-9c76-4785-b3ad-3791bfa1e28e"
+          (reference "#PWR02") (unit 1)
         )
       )
@@
         )
       )
+    )
+  )
+  (symbol (lib_id "power:+3V3") (at 203.2 87.63 0) (unit 1)
+    (in_bom yes) (on_board yes) (dnp no) (fields_autoplaced)
+    (property "Reference" "#PWR055" (at 203.2 91.44 0)
+      (effects (font (size 1.27 1.27)) hide)
+    )
+    (property "Value" "+3V3" (at 203.2 83.82 0)
+      (effects (font (size 1.27 1.27)))
+    )
+    (property "Footprint" "" (at 203.2 87.63 0)
+      (effects (font (size 1.27 1.27)) hide)
+    )
+    (property "Datasheet" "" (at 203.2 87.63 0)
+      (effects (font (size 1.27 1.27)) hide)
+    )
+    (pin "1")
+    (instances
+      (project "cwFOC"
+        (path "/ff847474-9801-42c6-af12-b4b1b75aa0af/50c76e34-9c76-4785-b3ad-3791bfa1e28e"
+          (reference "#PWR055") (unit 1)
+        )
+      )

Commit message: 完成第二版硬件
Parts:
- added D4: SMAJ15CA, Diode_SMD:D_SMA, symbol Device:D_TVS
Connections:
- net A+: now also J3.1 (Pin_1), D4.1 (A1); no longer J3.2 (Pin_2)
- net B-: now also J3.2 (Pin_2), D4.2 (A2); no longer J3.3 (Pin_3)
- net BRK: now also J3.3 (Pin_3); no longer J3.1 (Pin_1)
Changed lines of the file:
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@@
   (junction (at 165.1 87.63) (diameter 0) (color 0 0 0 0)
   )
+  (wire (pts (xy 165.1 87.63) (xy 179.07 87.63))
+    (stroke (width 0) (type default))
+  )
   (wire (pts (xy 151.13 87.63) (xy 165.1 87.63))
     (stroke (width 0) (type default))
   )
+  (wire (pts (xy 165.1 95.25) (xy 179.07 95.25))
+    (stroke (width 0) (type default))
+  )
   (wire (pts (xy 182.88 130.81) (xy 189.23 130.81))
     (stroke (width 0) (type default))
@@
     (stroke (width 0) (type default))
   )
+  (wire (pts (xy 184.15 123.19) (xy 189.23 123.19))
+    (stroke (width 0) (type default))
+  )
+  (wire (pts (xy 182.88 133.35) (xy 182.88 138.43))
+    (stroke (width 0) (type default))
+  )
+  (wire (pts (xy 177.8 128.27) (xy 189.23 128.27))
+    (stroke (width 0) (type default))
+  )
+  (wire (pts (xy 130.81 90.17) (xy 128.905 90.17))
+    (stroke (width 0) (type default))
+  )
   (wire (pts (xy 184.15 125.73) (xy 189.23 125.73))
-    (stroke (width 0) (type default))
-  )
-  (wire (pts (xy 182.88 133.35) (xy 182.88 138.43))
-    (stroke (width 0) (type default))
-  )
-  (wire (pts (xy 177.8 123.19) (xy 189.23 123.19))
-    (stroke (width 0) (type default))
-  )
-  (wire (pts (xy 130.81 90.17) (xy 128.905 90.17))
-    (stroke (width 0) (type default))
-  )
-  (wire (pts (xy 184.15 128.27) (xy 189.23 128.27))
     (stroke (width 0) (type default))
   )
@@
     (effects (font (size 1.27 1.27)) (justify left bottom))
   )
-  (label "B-" (at 184.15 128.27 0) (fields_autoplaced)
+  (label "B-" (at 184.15 125.73 0) (fields_autoplaced)
     (effects (font (size 1.27 1.27)) (justify left bottom))
   )
-  (label "A+" (at 184.15 125.73 0) (fields_autoplaced)
+  (label "A+" (at 184.15 123.19 0) (fields_autoplaced)
     (effects (font (size 1.27 1.27)) (justify left bottom))
   )
-  (global_label "BRK" (shape input) (at 177.8 123.19 180) (fields_autoplaced)
+  (global_label "BRK" (shape input) (at 177.8 128.27 180) (fields_autoplaced)
     (effects (font (size 1.27 1.27)) (justify right))
-    (property "Intersheetrefs" "${INTERSHEET_REFS}" (at 171.0842 123.19 0)
+    (property "Intersheetrefs" "${INTERSHEET_REFS}" (at 171.0842 128.27 0)
       (effects (font (size 1.27 1.27)) (justify right) hide)
     )
@@
         )
       )
+    )
+  )
+  (symbol (lib_id "Device:D_TVS") (at 179.07 91.44 90) (unit 1)
+    (in_bom yes) (on_board yes) (dnp no) (fields_autoplaced)
+    (property "Reference" "D4" (at 181.61 90.805 90)
+      (effects (font (size 1.27 1.27)) (justify right))
+    )
+    (property "Value" "SMAJ15CA" (at 181.61 93.345 90)
+      (effects (font (size 1.27 1.27)) (justify right))
+    )
+    (property "Footprint" "Diode_SMD:D_SMA" (at 179.07 91.44 0)
+      (effects (font (size 1.27 1.27)) hide)
+    )
+    (property "Datasheet" "~" (at 179.07 91.44 0)
+      (effects (font (size 1.27 1.27)) hide)
+    )
+    (pin "1")
+    (pin "2")
+    (instances
+      (project "cwFOC"
+        (path "/ff847474-9801-42c6-af12-b4b1b75aa0af/c3a6c5b4-78f3-47ea-a70d-c3f42438cf04"
+          (reference "D4") (unit 1)
+        )
+        (path "/ff847474-9801-42c6-af12-b4b1b75aa0af/50c76e34-9c76-4785-b3ad-3791bfa1e28e"
+          (reference "D7") (unit 1)
+        )
+      )
